File: PCB_Ethernet-1Gbps-Spartan-6/Ethernet.kicad_sch (KiCad schematic)
At the start: 54 parts, among them J1 ARJM11B1-502-AB-EW2, J2 Conn_02x20_Odd_Even, J3 Conn_01x02_Pin, Q1 PMOS, U2 KSZ9031RNXCC, U3 LD1117S12TR_SOT223, Y1 25Mhz

Commit message: rev2
Parts:
- added C23, C24, C28: 0.1uF, Capacitor_SMD:C_0603_1608Metric_Pad1.08x0.95mm_HandSolder, symbol Device:C_Small
- added C25, C26, C27, C29: 10uF, Capacitor_SMD:C_1206_3216Metric_Pad1.33x1.80mm_HandSolder, symbol Device:C_Small_US
- added F3: 0, Resistor_SMD:R_0805_2012Metric_Pad1.20x1.40mm_HandSolder, symbol Device:R_Small_US
- renumbered D3 to 3V3, D4 to 5V1, R20 to F1, R21 to F2, R19 to JP1
Connections:
- net 1.2V: now also C29.1
- net 3.3V: now also C25.1
- net A1.2V: now also C26.1, C28.2
- net A3.3V: now also C27.1
- net GND: now also C23.1, C24.1, C25.2, C26.2, C27.2, C28.1, C29.2, F3.1; no longer J1.S1 (SHIELD), J1.S2 (SHIELD__1)
- new net AGND: C23.2, C24.2, F3.2, J1.S1 (SHIELD), J1.S2 (SHIELD__1)
