File: PCB_Ethernet-1Gbps-Spartan-6/PCB_Ethernet-1Gbps-Spartan-6.kicad_pcb (KiCad board)
At the start: 2 copper layers, 54 x 47.5 mm, 71 parts, among them J1 ARJM11B1-502-AB-EW2, J2 Conn_02x20_Odd_Even, J3 Conn_01x02_Pin, Q1 PMOS, U2 KSZ9031RNXCC, U3 LD1117S12TR_SOT223, Y1 25Mhz

Commit message: rev1
Parts:
- renumbered R20 to FE1, R21 to FE2, R19 to JP1
Routing:
- net TD1+: track 15.6 -> 10.9 mm

Commit message: rev2
Parts:
- added C23: 0.1uF, Capacitor_SMD:C_0603_1608Metric_Pad1.08x0.95mm_HandSolder, F.Cu at (94.1, 117.7)
- added C24: 0.1uF, Capacitor_SMD:C_0603_1608Metric_Pad1.08x0.95mm_HandSolder, F.Cu at (92.6, 117.7)
- added C25: 10uF, Capacitor_SMD:C_1206_3216Metric_Pad1.33x1.80mm_HandSolder, B.Cu at (91.1, 89.3)
- added C26: 10uF, Capacitor_SMD:C_1206_3216Metric_Pad1.33x1.80mm_HandSolder, B.Cu at (96.1, 107.7)
- added C27: 10uF, Capacitor_SMD:C_1206_3216Metric_Pad1.33x1.80mm_HandSolder, B.Cu at (113.2, 107.0)
- added C28: 0.1uF, Capacitor_SMD:C_0603_1608Metric_Pad1.08x0.95mm_HandSolder, B.Cu at (99.9, 101.0)
- added C29: 10uF, Capacitor_SMD:C_1206_3216Metric_Pad1.33x1.80mm_HandSolder, B.Cu at (91.6, 109.2)
- added F3: 0, Resistor_SMD:R_0805_2012Metric_Pad1.20x1.40mm_HandSolder, F.Cu at (93.8, 113.9)
- moved GND 14.5 mm to (80.0, 118.8)
- moved G*** 4.19 mm to (86.7, 109.5)
- moved G*** 3.90 mm to (86.7, 118.5)
- moved C13 1.04 mm to (107.9, 103.8)
- moved C14 1.00 mm to (100.9, 103.8)
- renumbered 5V to 5V1, FE1 to F1, FE2 to F2
Connections:
- J1 pad S1: GND -> AGND
- J1 pad S2: GND -> AGND
Routing:
- net AGND: track 0.00 -> 24.6 mm
- net LED2: track 32.5 -> 38.2 mm
- net A1.2V: track 30.4 -> 32.8 mm
- net 1.2V: track 126.2 -> 128.1 mm
- net LED1: track 31.8 -> 30.7 mm

Commit message: rev3 firmware added
Parts:
- added J4: Conn_01x01_Pin, Connector_PinHeader_2.54mm:PinHeader_1x01_P2.54mm_Vertical, B.Cu at (115.4, 89.2)
- renumbered 5V1 to 5V0
Connections:
- J2 pad 11: unconnected-(J2-Pin_11-Pad11) -> Net-(J2-Pin_11)
- J2 pad 21: RXD1 -> RX_CLK
- J2 pad 23: RXD0 -> RXD1
- J2 pad 25: RX_DV -> RXD0
- J2 pad 27: RX_CLK -> RX_DV
Routing:
- net RX_CLK: track 16.0 -> 26.6 mm
- net RXD0: track 15.9 -> 26.5 mm
- net RX_DV: track 15.9 -> 26.5 mm
- net RXD1: track 16.1 -> 26.6 mm
- net RXD3: track 15.9 -> 24.4 mm
- net RXD2: track 15.9 -> 24.4 mm
- net Net-(J2-Pin_11): track 0.00 -> 2.33 mm
- net GND: vias 10 -> 9
Other:
- board text added: "RST_N 125Mhz INT_N MDIO MDC 3V3 RX_DV RXD0 RXD1 RX_CLK RXD2 RXD3 TX_EN GTX_CLK TXD3 TXD2 TXD1 TXD0 5V"
- board text removed: "RST_N 125Mhz INT_N MDIO MDC 3V3 RX_CLK RX_DV RXD0 RXD1 RXD2 RXD3 TX_EN GTX_CLK NC TXD3 TXD2 TXD1 TXD0 5V"

Commit message: mdio-and_uart_control_added
Parts:
- moved G*** 2.07 mm to (122.1, 114.2)
Changed lines of the file:
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@@
 		(tags "Through hole pin header THT 1x01 2.54mm single row")
 		(property "Reference" "J4"
-			(at 0 -2.2 -0)
+			(at 0 -2.2 0)
 			(layer "F.SilkS")
 			(effects
@@
 	(footprint "LOGO"
 		(layer "B.Cu")
-		(at 123.975 113.325 180)
+		(at 122.1 114.2 180)
 		(property "Reference" "G***"
 			(at 0 0 0)
@@
 		(last_track_width 0.3)
 		(last_tuning "24.5000 mm (tuned)")
-		(max_amplitude 2.05)
+		(max_amplitude 2.049999)
 		(min_amplitude 0.2)
 		(min_spacing 0.6)
